File: customKeyboard.kicad_pcb (KiCad board)
At the start: 2 copper layers, 158 parts, among them SW1 SW_Push, U1 ATmega32U4-AU, Y1 16MHz

Commit message: Placed Diode 1~11
Parts:
- moved D10 510.2 mm to (519.9, 40.5), turned to 90 degrees
- moved D11 429.2 mm to (539.0, 40.5), turned to 90 degrees
- moved MX27 352.9 mm to (540.5, 59.5)
- moved MX44 352.9 mm to (564.4, 78.6)
- moved MX56 352.9 mm to (516.7, 97.6)
- moved MX69 352.9 mm to (612.0, 116.7)
- moved D1 352.9 mm to (348.5, 40.5)
- moved D2 352.9 mm to (367.5, 40.5)
- moved D3 352.9 mm to (386.6, 40.5)
- moved D4 352.9 mm to (405.6, 40.5)
- moved D5 352.9 mm to (424.7, 40.5)
- moved MX1 352.9 mm to (340.5, 40.5)
- moved MX10 352.9 mm to (512.0, 40.5)
- moved MX11 352.9 mm to (531.0, 40.5)
- moved MX12 352.9 mm to (550.1, 40.5)
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Other:
- board outline added: 328.6 x 95.2 mm

Commit message: Placing complete and Replaced USB-C
Parts:
- removed USB1: Molex-0548190589, random-keyboard-parts:Molex-0548190589
- added J1: USB_C_Receptacle_USB2.0, Connector_USB:USB_C_Receptacle_Amphenol_12401548E4-2A, F.Cu at (618.3, 34.9)
- added R5: 5.1k, Resistor_SMD:R_0805_2012Metric, F.Cu at (617.4, 45.1)
- added R6: 5.1k, Resistor_SMD:R_0805_2012Metric, F.Cu at (620.3, 45.1)
- C1, C2, C3, C4, C5, C6, C7, F1, R1, R2, R3, R4, SW1, U1, Y1: moved to B.Cu
- moved D61 594.5 mm to (657.2, 97.6), turned to 90 degrees
- moved D60 569.9 mm to (638.2, 97.6), turned to 90 degrees
- moved D68 569.5 mm to (588.2, 116.7), turned to 90 degrees
- moved D67 535.1 mm to (565.1, 116.7), turned to 90 degrees
- moved D59 532.4 mm to (606.4, 100.8), turned to 90 degrees
- moved D16 520.6 mm to (657.2, 40.5), turned to 90 degrees
- moved D66 505.0 mm to (540.5, 116.7), turned to 90 degrees
- moved D15 496.7 mm to (638.2, 40.5), turned to 90 degrees
- moved D58 483.2 mm to (562.0, 97.6), turned to 90 degrees
- moved D13 475.8 mm to (576.3, 40.5), turned to 90 degrees
- moved D65 475.1 mm to (516.7, 120.7), turned to 90 degrees
- moved D57 458.7 mm to (542.9, 97.6), turned to 90 degrees
- moved D12 452.1 mm to (557.2, 40.5), turned to 90 degrees
- moved D31 440.4 mm to (638.2, 59.5), turned to 90 degrees
- moved C3 439.0 mm to (612.8, 69.2), turned to 90 degrees
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Connections:
- D14 pad 1: Net-(D14-Pad1) -> ROW3
- D19 pad 1: Net-(D19-Pad1) -> ROW3
- D24 pad 1: Net-(D24-Pad1) -> ROW3
- D29 pad 1: Net-(D29-Pad1) -> ROW3
- D34 pad 1: Net-(D34-Pad1) -> ROW3
- D39 pad 1: Net-(D39-Pad1) -> ROW3
- D4 pad 1: Net-(D4-Pad1) -> ROW3
- D44 pad 1: Net-(D44-Pad1) -> ROW3
- D49 pad 1: Net-(D49-Pad1) -> ROW3
- D54 pad 1: Net-(D54-Pad1) -> ROW3
- D58 pad 1: Net-(D58-Pad1) -> ROW3
- D62 pad 1: Net-(D62-Pad1) -> ROW3
- D66 pad 1: Net-(D66-Pad1) -> ROW3
- D9 pad 1: Net-(D9-Pad1) -> ROW3
- U1 pad 10: Net-(U1-Pad10) -> COL2
- U1 pad 11: Net-(U1-Pad11) -> COL3
- U1 pad 12: Net-(U1-Pad12) -> COL7
- U1 pad 18: Net-(U1-Pad18) -> COL10
- U1 pad 19: Net-(U1-Pad19) -> COL11
- U1 pad 20: Net-(U1-Pad20) -> COL12
- U1 pad 21: Net-(U1-Pad21) -> ROW4
- U1 pad 22: Net-(U1-Pad22) -> ROW2
- U1 pad 25: Net-(U1-Pad25) -> ROW3
- U1 pad 26: Net-(U1-Pad26) -> ROW1
- U1 pad 27: Net-(U1-Pad27) -> ROW0
- U1 pad 28: Net-(U1-Pad28) -> COL4
- U1 pad 29: Net-(U1-Pad29) -> COL5
- U1 pad 30: Net-(U1-Pad30) -> COL6
- U1 pad 31: Net-(U1-Pad31) -> COL8
- U1 pad 32: Net-(U1-Pad32) -> COL9
- U1 pad 39: Net-(U1-Pad39) -> COL15
- U1 pad 40: Net-(U1-Pad40) -> COL14
- U1 pad 41: Net-(U1-Pad41) -> COL13
- U1 pad 8: Net-(U1-Pad8) -> COL0
- U1 pad 9: Net-(U1-Pad9) -> COL1
Other:
- outline, holes or cut-outs redrawn
- net class Default: trace_width 0.25 -> 0.254
- net class Power added: clearance 0.2, trace_width 0.381, via_dia 0.8, via_drill 0.4

Commit message: ROW and COL0 complete
Parts:
- C1, C2: value 0.1uF -> 22pF
- C3: value 22pF -> 1uF
- C4: value 22pF -> 0.1uF
- C6: value 1uF -> 0.1uF
- MX13: footprint MX_Alps_Hybrid:MX-1U -> MX_Alps_Hybrid:MX-2.75U
- MX14: footprint MX_Alps_Hybrid:MX-2U -> MX_Alps_Hybrid:MX-1.25U
- MX15, MX31, MX60, MX61: footprint MX_Alps_Hybrid:MX-1U -> MX_Alps_Hybrid:MX-1.25U
- MX17: footprint MX_Alps_Hybrid:MX-1.5U -> MX_Alps_Hybrid:MX-1U
- MX20: footprint MX_Alps_Hybrid:MX-1U -> MX_Alps_Hybrid:MX-1.5U
- MX30: footprint MX_Alps_Hybrid:MX-1.5U -> MX_Alps_Hybrid:MX-1.25U
- MX33: footprint MX_Alps_Hybrid:MX-1.75U -> MX_Alps_Hybrid:MX-1U
- MX39: footprint MX_Alps_Hybrid:MX-1U -> MX_Alps_Hybrid:MX-1.75U
- MX42, MX70: footprint MX_Alps_Hybrid:MX-1U -> MX_Alps_Hybrid:MX-2.25U
- MX45, MX48: footprint MX_Alps_Hybrid:MX-2.25U -> MX_Alps_Hybrid:MX-1U
- MX46: footprint MX_Alps_Hybrid:MX-1U -> MX_Alps_Hybrid:MX-6.25U
- MX50: footprint MX_Alps_Hybrid:MX-1U -> MX_Alps_Hybrid:MX-2U
- MX59: footprint MX_Alps_Hybrid:MX-2.75U -> MX_Alps_Hybrid:MX-1U
- MX62, MX63, MX64, MX66, MX68: footprint MX_Alps_Hybrid:MX-1.25U -> MX_Alps_Hybrid:MX-1U
- MX65: footprint MX_Alps_Hybrid:MX-6.25U -> MX_Alps_Hybrid:MX-1U
- MX67: footprint MX_Alps_Hybrid:MX-1.25U -> MX_Alps_Hybrid:MX-1.5U
- R1, R2: value 22 -> 5.1k
- R4: value 10k -> 22
- R5: value 5.1k -> 22
- R6: value 5.1k -> 10k
- moved R1 28.9 mm to (608.7, 105.4), turned to 135 degrees
- moved R4 26.4 mm to (623.1, 103.2), turned to 45 degrees
- moved R2 21.7 mm to (606.4, 96.0)
- moved C6 17.2 mm to (606.4, 92.1)
- moved R3 14.6 mm to (611.2, 86.5), turned to 180 degrees
- moved C4 14.3 mm to (615.2, 86.5), turned to 180 degrees
- moved C1 11.7 mm to (619.1, 83.3), turned to 180 degrees
- moved C2 11.2 mm to (619.1, 80.2), turned to 180 degrees
- moved C3 10.1 mm to (619.1, 77.0), turned to 180 degrees
- moved C7 9.20 mm to (623.9, 88.1), turned to 135 degrees
- moved Y1 8.55 mm to (613.6, 75.4)
- moved F1 7.53 mm to (618.3, 44.5)
- moved C5 6.80 mm to (619.1, 86.5), turned to 180 degrees
- moved R5 4.17 mm to (621.5, 44.5)
- moved R6 3.61 mm to (623.9, 44.5)
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Connections:
- C1 pad 1: +5V -> Net-(C1-Pad1)
- C2 pad 1: +5V -> Net-(C2-Pad1)
- C4 pad 1: Net-(C4-Pad1) -> +5V
- C6 pad 1: Net-(C6-Pad1) -> +5V
- D10 pad 1: ROW4 -> ROW0
- D12 pad 1: ROW1 -> ROW0
- D13 pad 1: ROW2 -> ROW0
- D14 pad 1: ROW3 -> ROW0
- D15 pad 1: ROW4 -> ROW0
- D18 pad 1: ROW2 -> ROW1
- D19 pad 1: ROW3 -> ROW1
- D2 pad 1: ROW1 -> ROW0
- D20 pad 1: ROW4 -> ROW1
- D21 pad 1: ROW0 -> ROW1
- D23 pad 1: ROW2 -> ROW1
- D24 pad 1: ROW3 -> ROW1
- D25 pad 1: ROW4 -> ROW1
- D26 pad 1: ROW0 -> ROW1
- D28 pad 1: ROW2 -> ROW1
- D29 pad 1: ROW3 -> ROW1
- D3 pad 1: ROW2 -> ROW0
- D30 pad 1: ROW4 -> ROW1
- D31 pad 1: ROW0 -> ROW1
- D34 pad 1: ROW3 -> ROW2
- D35 pad 1: ROW4 -> ROW2
- D36 pad 1: ROW0 -> ROW2
- D37 pad 1: ROW1 -> ROW2
- D39 pad 1: ROW3 -> ROW2
- D4 pad 1: ROW3 -> ROW0
- D40 pad 1: ROW4 -> ROW2
- D41 pad 1: ROW0 -> ROW2
- D42 pad 1: ROW1 -> ROW2
- D44 pad 1: ROW3 -> ROW2
- D45 pad 1: ROW4 -> ROW2
- D46 pad 1: ROW0 -> ROW2
- D47 pad 1: ROW1 -> ROW2
- D48 pad 1: ROW2 -> ROW3
- D5 pad 1: ROW4 -> ROW0
- D50 pad 1: ROW4 -> ROW3
- D51 pad 1: ROW0 -> ROW3
- D52 pad 1: ROW1 -> ROW3
- D53 pad 1: ROW2 -> ROW3
- D55 pad 1: ROW0 -> ROW3
- D56 pad 1: ROW1 -> ROW3
- D57 pad 1: ROW2 -> ROW3
- D59 pad 1: ROW0 -> ROW3
- D60 pad 1: ROW1 -> ROW3
- D61 pad 1: ROW2 -> ROW3
- D62 pad 1: ROW3 -> ROW4
- D63 pad 1: ROW0 -> ROW4
- D64 pad 1: ROW1 -> ROW4
- D65 pad 1: ROW2 -> ROW4
- D66 pad 1: ROW3 -> ROW4
- D67 pad 1: ROW0 -> ROW4
- D68 pad 1: ROW1 -> ROW4
- D69 pad 1: ROW2 -> ROW4
- D7 pad 1: ROW1 -> ROW0
- D70 pad 1: ROW0 -> ROW4
- D71 pad 1: ROW1 -> ROW4
- D8 pad 1: ROW2 -> ROW0
- D9 pad 1: ROW3 -> ROW0
- MX10 pad 1: COL1 -> COL9
- MX11 pad 1: COL2 -> COL10
- MX12 pad 1: COL2 -> COL11
- MX13 pad 1: COL2 -> COL12
- MX14 pad 1: COL2 -> COL13
- MX15 pad 1: COL2 -> COL14
- MX16 pad 1: COL3 -> COL15
- MX17 pad 1: COL3 -> COL0
- MX18 pad 1: COL3 -> COL1
- MX19 pad 1: COL3 -> COL2
- MX2 pad 1: COL0 -> COL1
- MX22 pad 1: COL4 -> COL5
- MX23 pad 1: COL4 -> COL6
- MX24 pad 1: COL4 -> COL7
- MX25 pad 1: COL4 -> COL8
- MX26 pad 1: COL5 -> COL9
- MX27 pad 1: COL5 -> COL10
- MX28 pad 1: COL5 -> COL11
- MX29 pad 1: COL5 -> COL12
- MX3 pad 1: COL0 -> COL2
- MX30 pad 1: COL5 -> COL13
- MX31 pad 1: COL6 -> COL14
- MX32 pad 1: COL6 -> COL15
- MX33 pad 1: COL6 -> COL0
- MX34 pad 1: COL6 -> COL1
- MX35 pad 1: COL6 -> COL2
- MX36 pad 1: COL7 -> COL3
- MX37 pad 1: COL7 -> COL4
- MX38 pad 1: COL7 -> COL5
- MX39 pad 1: COL7 -> COL6
- MX4 pad 1: COL0 -> COL3
- MX42 pad 1: COL8 -> COL9
- MX43 pad 1: COL8 -> COL10
- MX44 pad 1: COL8 -> COL11
- MX45 pad 1: COL8 -> COL12
- MX46 pad 1: COL9 -> COL13
- MX47 pad 1: COL9 -> Net-(MX47-Pad1)
- MX48 pad 1: COL9 -> COL0
- MX49 pad 1: COL9 -> COL1
- MX5 pad 1: COL0 -> COL4
- MX50 pad 1: COL9 -> COL2
- MX51 pad 1: COL10 -> COL3
- MX52 pad 1: COL10 -> COL4
- MX53 pad 1: COL10 -> COL5
- MX54 pad 1: COL10 -> COL6
- MX55 pad 1: COL11 -> COL7
- MX56 pad 1: COL11 -> COL8
- MX57 pad 1: COL11 -> COL9
- MX58 pad 1: COL11 -> COL10
- MX59 pad 1: COL12 -> COL11
- MX6 pad 1: COL1 -> COL5
- MX61 pad 1: COL12 -> COL13
- MX62 pad 1: COL12 -> COL0
- MX63 pad 1: COL13 -> COL1
- MX64 pad 1: COL13 -> COL2
- MX65 pad 1: COL13 -> COL3
- MX66 pad 1: COL13 -> COL4
- MX67 pad 1: COL14 -> COL5
- MX68 pad 1: COL14 -> COL6
- MX69 pad 1: Net-(MX69-Pad1) -> COL7
- MX7 pad 1: COL1 -> COL6
- MX70 pad 1: COL15 -> COL8
- MX71 pad 1: COL15 -> COL9
- MX8 pad 1: COL1 -> COL7
- MX9 pad 1: COL1 -> COL8
- R1 pad 1: Net-(R1-Pad1) -> GND
- R1 pad 2: D- -> Net-(J1-PadA5)
- R2 pad 1: Net-(R2-Pad1) -> GND
- R2 pad 2: D+ -> Net-(J1-PadB5)
- R4 pad 1: GND -> Net-(R4-Pad1)
- R4 pad 2: Net-(R4-Pad2) -> D+
- R5 pad 1: GND -> Net-(R5-Pad1)
- R5 pad 2: Net-(J1-PadA5) -> D-
- R6 pad 2: Net-(J1-PadB5) -> Net-(R6-Pad2)
- U1 pad 16: Net-(C4-Pad1) -> Net-(C2-Pad1)
- U1 pad 17: Net-(C3-Pad1) -> Net-(C1-Pad1)
- U1 pad 3: Net-(R1-Pad1) -> Net-(R5-Pad1)
- U1 pad 33: Net-(R4-Pad2) -> Net-(R6-Pad2)
- U1 pad 4: Net-(R2-Pad1) -> Net-(R4-Pad1)
- U1 pad 6: Net-(C6-Pad1) -> Net-(C3-Pad1)
- Y1 pad 1: Net-(C3-Pad1) -> Net-(C1-Pad1)
- Y1 pad 3: Net-(C4-Pad1) -> Net-(C2-Pad1)
Routing:
- net ROW0: track 0.00 -> 384.5 mm, vias 0 -> 1
- net ROW1: track 0.00 -> 372.5 mm, vias 0 -> 3
- net ROW4: track 0.00 -> 357.2 mm, vias 0 -> 2
- net ROW3: track 0.00 -> 327.1 mm, vias 0 -> 1
- net ROW2: track 0.00 -> 325.9 mm, vias 0 -> 3
- net COL13: track 0.00 -> 137.9 mm, vias 0 -> 1
- net COL0: track 0.00 -> 100.1 mm
- net +5V: track 0.00 -> 93.1 mm
- net D-: track 0.00 -> 75.4 mm, vias 0 -> 2
- net D+: track 0.00 -> 65.2 mm
- net Net-(R3-Pad2): track 0.00 -> 28.9 mm
- net Net-(C3-Pad1): track 0.00 -> 24.4 mm
- net Net-(D59-Pad2): track 0.00 -> 16.7 mm
- net VCC: track 0.00 -> 15.9 mm, vias 0 -> 2
- net Net-(C4-Pad1): track 0.00 -> 15.1 mm
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Other:
- copper layers 2 -> 4

Commit message: 80% Complete
Parts:
- MX13: footprint MX_Alps_Hybrid:MX-2.75U -> MX_Alps_Hybrid:MX-1U
- MX14: footprint MX_Alps_Hybrid:MX-1.25U -> MX_Alps_Hybrid:MX-2U
- MX15, MX31, MX60, MX61: footprint MX_Alps_Hybrid:MX-1.25U -> MX_Alps_Hybrid:MX-1U
- MX17: footprint MX_Alps_Hybrid:MX-1U -> MX_Alps_Hybrid:MX-1.5U
- MX20: footprint MX_Alps_Hybrid:MX-1.5U -> MX_Alps_Hybrid:MX-1U
- MX30: footprint MX_Alps_Hybrid:MX-1.25U -> MX_Alps_Hybrid:MX-1.5U
- MX33: footprint MX_Alps_Hybrid:MX-1U -> MX_Alps_Hybrid:MX-1.75U
- MX39: footprint MX_Alps_Hybrid:MX-1.75U -> MX_Alps_Hybrid:MX-1U
- MX42, MX70: footprint MX_Alps_Hybrid:MX-2.25U -> MX_Alps_Hybrid:MX-1U
- MX45, MX48: footprint MX_Alps_Hybrid:MX-1U -> MX_Alps_Hybrid:MX-2.25U
- MX46: footprint MX_Alps_Hybrid:MX-6.25U -> MX_Alps_Hybrid:MX-1U
- MX50: footprint MX_Alps_Hybrid:MX-2U -> MX_Alps_Hybrid:MX-1U
- MX59: footprint MX_Alps_Hybrid:MX-1U -> MX_Alps_Hybrid:MX-2.75U
- MX62, MX63, MX64, MX66, MX68: footprint MX_Alps_Hybrid:MX-1U -> MX_Alps_Hybrid:MX-1.25U
- MX65: footprint MX_Alps_Hybrid:MX-1U -> MX_Alps_Hybrid:MX-6.25U
- MX67: footprint MX_Alps_Hybrid:MX-1.5U -> MX_Alps_Hybrid:MX-1.25U
- moved R4 19.1 mm to (609.6, 89.7)
Connections:
- MX47 pad 1: Net-(MX47-Pad1) -> COL14
Routing:
- net COL1: track 0.00 -> 340.2 mm, vias 0 -> 2
- net COL3: track 0.00 -> 323.2 mm, vias 0 -> 2
- net COL2: track 0.00 -> 319.3 mm, vias 0 -> 2
- net COL4: track 0.00 -> 287.4 mm, vias 0 -> 2
- net COL0: track 100.1 -> 380.3 mm, vias 0 -> 1
- net COL5: track 0.00 -> 265.5 mm, vias 0 -> 3
- net COL6: track 0.00 -> 240.7 mm, vias 0 -> 2
- net COL7: track 0.00 -> 222.3 mm, vias 0 -> 2
- net COL8: track 0.00 -> 212.8 mm, vias 0 -> 2
- net COL9: track 0.00 -> 212.2 mm, vias 0 -> 1
- net COL14: track 0.00 -> 97.7 mm
- net COL15: track 0.00 -> 84.8 mm
- net COL11: track 0.00 -> 82.2 mm
- net COL10: track 0.00 -> 68.3 mm
- net Net-(J1-PadA5): track 4.57 -> 71.3 mm, vias 0 -> 4
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
Commit message: Complete!
Routing:
- net COL12: track 50.0 -> 147.0 mm
- net COL10: track 68.3 -> 144.2 mm, vias 0 -> 1
- net COL11: track 82.2 -> 120.6 mm, vias 0 -> 1
- net GND: track 0.00 -> 32.4 mm
- net +5V: track 94.7 -> 110.8 mm, vias 0 -> 2
- net ROW0: track 389.9 -> 397.0 mm
- net Net-(C1-Pad1): track 23.7 -> 24.1 mm, vias 0 -> 2
- added copper zone on F.Cu, net +5V
- added copper zone on B.Cu, net GND
Other:
- board size 328.6 x 95.2 mm -> 328.6 x 97.8 mm
- board text added: "α-60 PCB V1 2022-12-02"
